File: MapleMini/MapleMini.sch (KiCad schematic (older format))
At the start: 39 parts

Commit message: Updates after re-oopening in KiCAD 5.1.7
Parts:
- J?: symbol Connector:USB_C_Receptacle_USB2.0 -> MapleMini-rescue:USB_C_Receptacle_USB2.0-Connector
Changed lines of the file:
@@
 $EndDescr
 $Comp
-L Connector:USB_C_Receptacle_USB2.0 J?
+L MapleMini-rescue:USB_C_Receptacle_USB2.0-Connector J?
 U 1 1 5F56CB65
 P 1000 1550
