File: project files/derived from Baite/MapleMini.kicad_pcb (KiCad board)
At the start: 2 copper layers, 51.1 x 18 mm, 36 parts, among them J1 USB_C, J2 Left, J3 Right, Q1 BC817, Q2 BC817, SW1 Reset, SW2 Button, U1 STM32F103CBTx, U2 AMS1117-3.3, Y1 8MHz

Commit message: Added STDC connectors
Parts:
- added J2: Conn_ST_STDC14, Connector_PinHeader_1.27mm:PinHeader_2x07_P1.27mm_Vertical_SMD, F.Cu at (94.6, 85.1)
- renumbered D2 to D1, D1 to D2, J2 to J3, J3 to J4, R14 to R12, R12 to R13, R13 to R14, R3 to R2, R2 to R3, R5 to R4, R6 to R5, R4 to R6, R8 to R7, R7 to R8
Connections:
- net /19 renamed SWO
- net /21 renamed SWCLK
- net /22 renamed SWDIO
- net /25 renamed RX
- net /26 renamed TX
